File: ContadorDePasajeros.sch (KiCad schematic (older format))
At the start: 13 parts, among them J1 Conector_in, J3 Conector_esp, U1 ESP01

Commit message: Serigrafia, agujeros y ajustes
Parts:
- added MH1, MH2, MH3, MH4: MountingHole, Mounting_Holes:MountingHole_2.5mm, symbol Mechanical:MountingHole
Changed lines of the file:
@@
 	1750 950  2100 950
 Connection ~ 2100 950
+$Comp
+L Mechanical:MountingHole MH1
+U 1 1 5BC3B7D1
+P 6300 2800
+F 0 "MH1" H 6400 2846 50  0000 L CNN
+F 1 "MountingHole" H 6400 2755 50  0000 L CNN
+F 2 "Mounting_Holes:MountingHole_2.5mm" H 6300 2800 50  0001 C CNN
+F 3 "~" H 6300 2800 50  0001 C CNN
+	1    6300 2800
+	1    0    0    -1
+$EndComp
+$Comp
+L Mechanical:MountingHole MH2
+U 1 1 5BC3B8C5
+P 6300 3000
+F 0 "MH2" H 6400 3046 50  0000 L CNN
+F 1 "MountingHole" H 6400 2955 50  0000 L CNN
+F 2 "Mounting_Holes:MountingHole_2.5mm" H 6300 3000 50  0001 C CNN
+F 3 "~" H 6300 3000 50  0001 C CNN
+	1    6300 3000
+	1    0    0    -1
+$EndComp
+$Comp
+L Mechanical:MountingHole MH3
+U 1 1 5BC3B905
+P 6300 3200
+F 0 "MH3" H 6400 3246 50  0000 L CNN
+F 1 "MountingHole" H 6400 3155 50  0000 L CNN
+F 2 "Mounting_Holes:MountingHole_2.5mm" H 6300 3200 50  0001 C CNN
+F 3 "~" H 6300 3200 50  0001 C CNN
+	1    6300 3200
+	1    0    0    -1
+$EndComp
+$Comp
+L Mechanical:MountingHole MH4
+U 1 1 5BC3B939
+P 6300 3400
+F 0 "MH4" H 6400 3446 50  0000 L CNN
+F 1 "MountingHole" H 6400 3355 50  0000 L CNN
+F 2 "Mounting_Holes:MountingHole_2.5mm" H 6300 3400 50  0001 C CNN
+F 3 "~" H 6300 3400 50  0001 C CNN
+	1    6300 3400
+	1    0    0    -1
+$EndComp
 $EndSCHEMATC

Commit message: Correcciones adrian
Parts:
- MH1: value MountingHole -> MH1
- MH2: value MountingHole -> MH2
- MH3: value MountingHole -> MH3
- MH4: value MountingHole -> MH4
Changed lines of the file:
@@
 U 1 1 5BB23C65
 P 4450 2350
-F 0 "Rx_up1" H 4520 2396 50  0000 L CNN
-F 1 "1k" H 4520 2305 50  0000 L CNN
+F 0 "Rx_up1" V 4550 2200 50  0000 L CNN
+F 1 "1k" V 4350 2300 50  0000 L CNN
 F 2 "Resistor_SMD:R_0805_2012Metric_Pad1.15x1.40mm_HandSolder" V 4380 2350 50  0001 C CNN
 F 3 "~" H 4450 2350 50  0001 C CNN
@@
 L Device:C C_F1
 U 1 1 5BBE4CB7
-P 1750 1900
-F 0 "C_F1" H 1865 1946 50  0000 L CNN
-F 1 "100n" H 1865 1855 50  0000 L CNN
-F 2 "Capacitor_THT:CP_Radial_Tantal_D4.5mm_P5.00mm" H 1788 1750 50  0001 C CNN
-F 3 "~" H 1750 1900 50  0001 C CNN
-	1    1750 1900
-	1    0    0    -1
-$EndComp
-Wire Wire Line
-	2100 2750 1750 2750
-Wire Wire Line
-	1750 2750 1750 2050
-Wire Wire Line
-	1750 1750 1750 950
-Wire Wire Line
-	1750 950  2100 950
+P 1650 1900
+F 0 "C_F1" H 1765 1946 50  0000 L CNN
+F 1 "100n" H 1765 1855 50  0000 L CNN
+F 2 "Capacitor_THT:CP_Radial_Tantal_D4.5mm_P5.00mm" H 1688 1750 50  0001 C CNN
+F 3 "~" H 1650 1900 50  0001 C CNN
+	1    1650 1900
+	1    0    0    -1
+$EndComp
+Wire Wire Line
+	2100 2750 1650 2750
+Wire Wire Line
+	1650 2750 1650 2050
+Wire Wire Line
+	1650 1750 1650 950
+Wire Wire Line
+	1650 950  2100 950
 Connection ~ 2100 950
 $Comp
@@
 P 6300 2800
 F 0 "MH1" H 6400 2846 50  0000 L CNN
-F 1 "MountingHole" H 6400 2755 50  0000 L CNN
+F 1 "MH1" H 6400 2755 50  0000 L CNN
 F 2 "Mounting_Holes:MountingHole_2.5mm" H 6300 2800 50  0001 C CNN
 F 3 "~" H 6300 2800 50  0001 C CNN
@@
 P 6300 3000
 F 0 "MH2" H 6400 3046 50  0000 L CNN
-F 1 "MountingHole" H 6400 2955 50  0000 L CNN
+F 1 "MH2" H 6400 2955 50  0000 L CNN
 F 2 "Mounting_Holes:MountingHole_2.5mm" H 6300 3000 50  0001 C CNN
 F 3 "~" H 6300 3000 50  0001 C CNN
@@
 P 6300 3200
 F 0 "MH3" H 6400 3246 50  0000 L CNN
-F 1 "MountingHole" H 6400 3155 50  0000 L CNN
+F 1 "MH3" H 6400 3155 50  0000 L CNN
 F 2 "Mounting_Holes:MountingHole_2.5mm" H 6300 3200 50  0001 C CNN
 F 3 "~" H 6300 3200 50  0001 C CNN
@@
 P 6300 3400
 F 0 "MH4" H 6400 3446 50  0000 L CNN
-F 1 "MountingHole" H 6400 3355 50  0000 L CNN
+F 1 "MH4" H 6400 3355 50  0000 L CNN
 F 2 "Mounting_Holes:MountingHole_2.5mm" H 6300 3400 50  0001 C CNN
 F 3 "~" H 6300 3400 50  0001 C CNN

Commit message: Power flag agregado
Connections:
- wire segments 63 -> 67
Changed lines of the file:
@@
 L Connector:Conn_01x04_Female J1
 U 1 1 5BB1C2B8
-P 6350 750
-F 0 "J1" H 6377 726 50  0000 L CNN
-F 1 "Conector_in" H 6377 635 50  0000 L CNN
-F 2 "Connector_PinSocket_2.54mm:PinSocket_1x04_P2.54mm_Vertical" H 6350 750 50  0001 C CNN
-F 3 "~" H 6350 750 50  0001 C CNN
-	1    6350 750
-	1    0    0    -1
-$EndComp
-Text GLabel 5900 650  0    50   BiDi ~ 0
+P 6800 800
+F 0 "J1" H 6827 776 50  0000 L CNN
+F 1 "Conector_in" H 6827 685 50  0000 L CNN
+F 2 "Connector_PinSocket_2.54mm:PinSocket_1x04_P2.54mm_Vertical" H 6800 800 50  0001 C CNN
+F 3 "~" H 6800 800 50  0001 C CNN
+	1    6800 800
+	1    0    0    -1
+$EndComp
+Text GLabel 6350 700  0    50   BiDi ~ 0
 Rx
-Text GLabel 5900 750  0    50   BiDi ~ 0
+Text GLabel 6350 800  0    50   BiDi ~ 0
 Tx
 Wire Wire Line
-	6150 650  5900 650
-Wire Wire Line
-	5900 750  6150 750
+	6600 700  6350 700
+Wire Wire Line
+	6350 800  6600 800
 $Comp
 L power:+3.3V #PWR0108
 U 1 1 5BB1EB83
-P 5850 850
-F 0 "#PWR0108" H 5850 700 50  0001 C CNN
-F 1 "+3.3V" H 5865 1023 50  0000 C CNN
-F 2 "" H 5850 850 50  0001 C CNN
-F 3 "" H 5850 850 50  0001 C CNN
-	1    5850 850
+P 5900 900
+F 0 "#PWR0108" H 5900 750 50  0001 C CNN
+F 1 "+3.3V" H 5915 1073 50  0000 C CNN
+F 2 "" H 5900 900 50  0001 C CNN
+F 3 "" H 5900 900 50  0001 C CNN
+	1    5900 900
 	0    -1   -1   0
 $EndComp
@@
 L power:GND #PWR0109
 U 1 1 5BB1ED0A
-P 5900 950
-F 0 "#PWR0109" H 5900 700 50  0001 C CNN
-F 1 "GND" H 5905 777 50  0000 C CNN
-F 2 "" H 5900 950 50  0001 C CNN
-F 3 "" H 5900 950 50  0001 C CNN
-	1    5900 950
-	1    0    0    -1
-$EndComp
-Wire Wire Line
-	6150 950  5900 950
-Wire Wire Line
-	5850 850  6150 850
+P 6200 1000
+F 0 "#PWR0109" H 6200 750 50  0001 C CNN
+F 1 "GND" H 6205 827 50  0000 C CNN
+F 2 "" H 6200 1000 50  0001 C CNN
+F 3 "" H 6200 1000 50  0001 C CNN
+	1    6200 1000
+	0    1    1    0
+$EndComp
+Wire Wire Line
+	6600 1000 6300 1000
+Wire Wire Line
+	5900 900  6050 900
 Wire Wire Line
 	4750 2900 4750 2800
@@
 	1    0    0    -1
 $EndComp
+$Comp
+L power:PWR_FLAG #FLG0101
+U 1 1 5BCAA10C
+P 6050 800
+F 0 "#FLG0101" H 6050 875 50  0001 C CNN
+F 1 "PWR_FLAG" H 6050 974 50  0000 C CNN
+F 2 "" H 6050 800 50  0001 C CNN
+F 3 "~" H 6050 800 50  0001 C CNN
+	1    6050 800
+	1    0    0    -1
+$EndComp
+Wire Wire Line
+	6050 800  6050 900
+Connection ~ 6050 900
+Wire Wire Line
+	6050 900  6600 900
+$Comp
+L power:PWR_FLAG #FLG0102
+U 1 1 5BCAD9D4
+P 6300 1100
+F 0 "#FLG0102" H 6300 1175 50  0001 C CNN
+F 1 "PWR_FLAG" H 6300 1273 50  0000 C CNN
+F 2 "" H 6300 1100 50  0001 C CNN
+F 3 "~" H 6300 1100 50  0001 C CNN
+	1    6300 1100
+	-1   0    0    1
+$EndComp
+Wire Wire Line
+	6300 1100 6300 1000
+Connection ~ 6300 1000
+Wire Wire Line
+	6300 1000 6200 1000
 $EndSCHEMATC
